File: SCH-PCB/EAGLE/i2c_relay.brd (EAGLE design)
At the start: 49.5 x 97.1 mm, 71 parts, among them IC1 PCF8575TS_1,118, Q1 MMST2222A-7-F, Q2 MMST2222A-7-F, Q3 MMST2222A-7-F, Q4 MMST2222A-7-F, Q5 MMST2222A-7-F, Q6 MMST2222A-7-F, Q7 MMST2222A-7-F, Q8 MMST2222A-7-F

Commit message: FEAT: update silkscreen board pcb
Routing:
- net GND: vias 55 -> 56
Other:
- outline, holes or cut-outs redrawn
- board text added: "5V"
- board text added: "A0"
- board text added: "A1"
- board text added: "A2"
- board text added: "COM"
- board text added: "GND"
- board text added: "INT"
- board text added: "NO"
- board text added: "RELAY 1"
- board text added: "RELAY 2"
- board text added: "RELAY 3"
- board text added: "RELAY 4"
- board text added: "RELAY 5"
- board text added: "RELAY 6"
- board text added: "RELAY 7"
- board text added: "RELAY 8"
- board text added: "SCL"
- board text added: "SDA"
- board text added: "VCC"
